File: Uguisu.kicad_sch (KiCad schematic)
At the start: 8 parts, among them U1 XIAO-nRF52840-SMD

Commit message: README: GPIO table with LED1 pin 4,5,6 in notes
Made-with: Cursor
Parts:
- renumbered LED2 to LED1, R3 to R1, R1 to R2, R2 to R3
Connections:
- net MCU_D1: now also R1.2; no longer R3.1
- net MCU_D3: now also R3.1; no longer R1.2
Changed lines of the file:
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@@
 		)
 	)
-	(label "MCU_D1"
+	(label "MCU_D3"
 		(at 162.56 86.36 0)
 		(effects
@@
 		)
 	)
-	(label "MCU_D3"
+	(label "MCU_D1"
 		(at 162.56 96.52 0)
 		(effects
@@
 		(on_board yes)
 		(dnp no)
-		(property "Reference" "LED2"
+		(property "Reference" "LED1"
 			(at 150.62 77.47 0)
 			(effects
@@
 			(project ""
 				(path "/3411fae6-0f44-4a47-8bb3-5970407324d6"
-					(reference "LED2")
+					(reference "LED1")
 					(unit 1)
 				)
@@
 		(on_board yes)
 		(dnp no)
-		(property "Reference" "R3"
+		(property "Reference" "R1"
 			(at 158.75 94.488 90)
 			(effects
@@
 			(project ""
 				(path "/3411fae6-0f44-4a47-8bb3-5970407324d6"
-					(reference "R3")
+					(reference "R1")
 					(unit 1)
 				)
@@
 		(on_board yes)
 		(dnp no)
-		(property "Reference" "R1"
+		(property "Reference" "R2"
 			(at 158.75 89.408 90)
 			(effects
@@
 			(project ""
 				(path "/3411fae6-0f44-4a47-8bb3-5970407324d6"
-					(reference "R1")
+					(reference "R2")
 					(unit 1)
 				)
@@
 		(on_board yes)
 		(dnp no)
-		(property "Reference" "R2"
+		(property "Reference" "R3"
 			(at 158.75 84.328 90)
 			(effects
@@
 			(project ""
 				(path "/3411fae6-0f44-4a47-8bb3-5970407324d6"
-					(reference "R2")
-					(unit 1)
-				)
+					(reference "R3")
+					(unit 1)
+				)
