File: Uguisu.kicad_pcb (KiCad board)
At the start: 2 copper layers, 35 x 50 mm, 8 parts, among them U1 XIAO-nRF52840-SMD

Commit message: Update PCB layout
Made-with: Cursor
Parts:
- renumbered LED2 to LED1, R3 to R1, R1 to R2, R2 to R3
Connections:
- R1 pad 2: /MCU_D3 -> /MCU_D1
- R2 pad 2: /MCU_D1 -> /MCU_D2
- R3 pad 1: /MCU_D2 -> /MCU_D3
Routing:
- net /MCU_D2: track 0.00 -> 18.0 mm
- net /MCU_D1: track 0.02 -> 17.3 mm
- net /MCU_D3: track 0.00 -> 16.4 mm
- net +BATT: track 12.7 -> 20.2 mm
Changed lines of the file:
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@@
 	(net 14 "/MCU_D2")
 	(net 15 "/MCU_D3")
-	(net 16 "Net-(LED2---Pad4)")
-	(net 17 "Net-(LED2---Pad6)")
-	(net 18 "Net-(LED2---Pad5)")
+	(net 16 "Net-(LED1---Pad4)")
+	(net 17 "Net-(LED1---Pad6)")
+	(net 18 "Net-(LED1---Pad5)")
 	(footprint "Seeed_Studio_XIAO_Series:XIAO-nRF52840-SMD"
 		(layer "F.Cu")
@@
 		(layer "B.Cu")
 		(at 119.25 76)
-		(property "Reference" "LED2"
+		(property "Reference" "LED1"
 			(at 0 5.5 0)
 			(layer "B.SilkS")
@@
 			(size 2.26 1)
 			(layers "B.Cu" "B.Mask" "B.Paste")
-			(net 16 "Net-(LED2---Pad4)")
+			(net 16 "Net-(LED1---Pad4)")
 			(pinfunction "-")
 			(pintype "unspecified")
@@
 			(size 2.26 1)
 			(layers "B.Cu" "B.Mask" "B.Paste")
-			(net 18 "Net-(LED2---Pad5)")
+			(net 18 "Net-(LED1---Pad5)")
 			(pinfunction "-")
 			(pintype "unspecified")
@@
 			(size 2.26 1)
 			(layers "B.Cu" "B.Mask" "B.Paste")
-			(net 17 "Net-(LED2---Pad6)")
+			(net 17 "Net-(LED1---Pad6)")
 			(pinfunction "-")
 			(pintype "unspecified")
@@
 		(descr "Resistor SMD 0603 (1608 Metric), square (rectangular) end terminal, IPC-7351 nominal, (Body size source: IPC-SM-782 page 72, https://www.pcb-3d.com/wordpress/wp-content/uploads/ipc-sm-782a_amendment_1_and_2.pdf), generated with kicad-footprint-generator")
 		(tags "resistor")
-		(property "Reference" "R3"
+		(property "Reference" "R1"
 			(at 0 1.43 0)
 			(layer "B.SilkS")
@@
 			(layers "B.Cu" "B.Mask" "B.Paste")
 			(roundrect_rratio 0.25)
-			(net 16 "Net-(LED2---Pad4)")
+			(net 16 "Net-(LED1---Pad4)")
 			(pintype "passive")
 		)
@@
 			(layers "B.Cu" "B.Mask" "B.Paste")
 			(roundrect_rratio 0.25)
-			(net 15 "/MCU_D3")
+			(net 1 "/MCU_D1")
 			(pintype "passive")
 		)
@@
 		(descr "Resistor SMD 0603 (1608 Metric), square (rectangular) end terminal, IPC-7351 nominal, (Body size source: IPC-SM-782 page 72, https://www.pcb-3d.com/wordpress/wp-content/uploads/ipc-sm-782a_amendment_1_and_2.pdf), generated with kicad-footprint-generator")
 		(tags "resistor")
-		(property "Reference" "R1"
+		(property "Reference" "R2"
 			(at 0 1.43 0)
 			(layer "B.SilkS")
@@
 			(layers "B.Cu" "B.Mask" "B.Paste")
 			(roundrect_rratio 0.25)
-			(net 18 "Net-(LED2---Pad5)")
+			(net 18 "Net-(LED1---Pad5)")
 			(pintype "passive")
 		)
@@
 			(layers "B.Cu" "B.Mask" "B.Paste")
 			(roundrect_rratio 0.25)
-			(net 1 "/MCU_D1")
+			(net 14 "/MCU_D2")
 			(pintype "passive")
 		)
@@
 		(descr "Resistor SMD 0603 (1608 Metric), square (rectangular) end terminal, IPC-7351 nominal, (Body size source: IPC-SM-782 page 72, https://www.pcb-3d.com/wordpress/wp-content/uploads/ipc-sm-782a_amendment_1_and_2.pdf), generated with kicad-footprint-generator")
 		(tags "resistor")
-		(property "Reference" "R2"
+		(property "Reference" "R3"
 			(at 0 1.43 0)
 			(layer "B.SilkS")
@@
 			(layers "B.Cu" "B.Mask" "B.Paste")
 			(roundrect_rratio 0.25)
-			(net 14 "/MCU_D2")
+			(net 15 "/MCU_D3")
 			(pintype "passive")
 		)
@@
 			(layers "B.Cu" "B.Mask" "B.Paste")
 			(roundrect_rratio 0.25)
-			(net 17 "Net-(LED2---Pad6)")
+			(net 17 "Net-(LED1---Pad6)")
 			(pintype "passive")
 		)
@@
 		(layer "Edge.Cuts")
 	)
+	(segment
+		(start 124.75 74.5)
+		(end 116.55 66.3)
+		(width 0.5)
+		(layer "F.Cu")
+		(net 1)
+	)
+	(segment
+		(start 116.55 66.3)
+		(end 110.835 66.3)
+		(width 0.5)
+		(layer "F.Cu")
+		(net 1)
+	)
 	(via
-		(at 124.75 76)
+		(at 124.75 74.5)
 		(size 0.6)
 		(drill 0.3)
@@
 		(start 114.445 69.155)
 		(end 114.45 69.15)
-		(width 0.5)
-		(layer "F.Cu")
-		(net 2)
-	)
-	(segment
-		(start 115.9 87.6)
-		(end 122.1 87.6)
 		(width 0.5)
 		(layer "F.Cu")
@@
 	)
 	(segment
+		(start 122.1 87.6)
+		(end 115.9 87.6)
+		(width 0.5)
+		(layer "B.Cu")
+		(net 2)
+	)
+	(segment
 		(start 114.4235 71.0665)
 		(end 114.41 71.08)
@@
 	)
 	(segment
+		(start 117.04 74.5)
+		(end 117.04 73.6615)
+		(width 0.5)
+		(layer "B.Cu")
+		(net 12)
+	)
+	(segment
+		(start 117.04 76)
+		(end 117.04 77.5)
+		(width 0.5)
+		(layer "B.Cu")
+		(net 12)
+	)
+	(segment
+		(start 117.04 74.5)
+		(end 117.04 76)
+		(width 0.5)
+		(layer "B.Cu")
+		(net 12)
+	)
+	(segment
 		(start 105.5 80)
 		(end 105.5115 80)
@@
 	)
 	(segment
+		(start 117.04 73.6615)
+		(end 114.445 71.0665)
+		(width 0.5)
+		(layer "B.Cu")
+		(net 12)
+	)
+	(segment
 		(start 108.375 65.875)
 		(end 110.49 63.76)
-		(width 0.5)
-		(layer "F.Cu")
-		(net 13)
-	)
-	(segment
-		(start 115.9 83.9)
-		(end 122.1 83.9)
 		(width 0.5)
 		(layer "F.Cu")
@@
 		(net 13)
 	)
+	(segment
+		(start 115.9 83.9)
+		(end 122.1 83.9)
+		(width 0.5)
+		(layer "B.Cu")
+		(net 13)
+	)
+	(segment
+		(start 124.75 76)
+		(end 116.25 67.5)
+		(width 0.5)
+		(layer "F.Cu")
+		(net 14)
+	)
+	(segment
+		(start 111.924 67.751)
+		(end 110.835 68.84)
+		(width 0.5)
+		(layer "F.Cu")
+		(net 14)
+	)
+	(segment
+		(start 112.11119 67.751)
+		(end 111.924 67.751)
+		(width 0.5)
+		(layer "F.Cu")
+		(net 14)
+	)
+	(segment
+		(start 116.25 67.5)
+		(end 112.36219 67.5)
+		(width 0.5)
+		(layer "F.Cu")
+		(net 14)
+	)
+	(segment
+		(start 112.36219 67.5)
+		(end 112.11119 67.751)
+		(width 0.5)
+		(layer "F.Cu")
+		(net 14)
+	)
+	(via
+		(at 124.75 76)
+		(size 0.6)
+		(drill 0.3)
+		(layers "F.Cu" "B.Cu")
+		(net 14)
+	)
+	(segment
+		(start 119.719 72.469)
+		(end 111.924 72.469)
+		(width 0.5)
+		(layer "F.Cu")
+		(net 15)
+	)
+	(segment
+		(start 111.924 72.469)
+		(end 110.835 71.38)
+		(width 0.5)
+		(layer "F.Cu")
+		(net 15)
+	)
+	(segment
+		(start 124.75 77.5)
+		(end 119.719 72.469)
+		(width 0.5)
+		(layer "F.Cu")
+		(net 15)
+	)
 	(via
 		(at 124.75 77.5)
 		(size 0.6)
 		(drill 0.3)
-		(layers "F.Cu" "B.Cu")
-		(net 14)
-	)
-	(via
-		(at 124.75 74.5)
-		(size 0.6)
-		(drill 0.3)

Commit message: README and PCB updates
Made-with: Cursor
Routing:
- net +BATT: track 20.2 -> 28.3 mm
Changed lines of the file:
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@@
 	)
 	(gr_line
-		(start 103.5 60.75)
-		(end 134.5 60.75)
+		(start 103.525 60.75)
+		(end 134.525 60.75)
 		(stroke
 			(width 0.2)
@@
 	)
 	(gr_line
-		(start 136.5 62.75)
-		(end 136.5 108.75)
+		(start 136.525 62.75)
+		(end 136.525 108.75)
 		(stroke
 			(width 0.2)
@@
 	)
 	(gr_circle
-		(center 105.25 106.99985)
-		(end 106.38 108.64985)
+		(center 105.275 106.99985)
+		(end 106.405 108.64985)
 		(stroke
 			(width 0.2)
@@
 	)
 	(gr_arc
-		(start 103.5 110.75)
-		(mid 102.085786 110.164214)
-		(end 101.5 108.75)
+		(start 103.525 110.75)
+		(mid 102.110786 110.164214)
+		(end 101.525 108.75)
 		(stroke
 			(width 0.2)
@@
 	)
 	(gr_arc
-		(start 134.5 60.75)
-		(mid 135.914214 61.335786)
-		(end 136.5 62.75)
+		(start 134.525 60.75)
+		(mid 135.939214 61.335786)
+		(end 136.525 62.75)
 		(stroke
 			(width 0.2)
@@
 	)
 	(gr_line
-		(start 101.5 108.75)
-		(end 101.5 62.75)
+		(start 101.525 108.75)
+		(end 101.525 62.75)
 		(stroke
 			(width 0.2)
@@
 	)
 	(gr_line
-		(start 134.5 110.75)
-		(end 103.5 110.75)
+		(start 134.525 110.75)
+		(end 103.525 110.75)
 		(stroke
 			(width 0.2)
@@
 	)
 	(gr_arc
-		(start 101.5 62.75)
-		(mid 102.085786 61.335786)
-		(end 103.5 60.75)
+		(start 101.525 62.75)
+		(mid 102.110786 61.335786)
+		(end 103.525 60.75)
 		(stroke
 			(width 0.2)
@@
 	)
 	(gr_circle
-		(center 105.25 64.49955)
-		(end 106.38 66.14955)
+		(center 105.275 64.49955)
+		(end 106.405 66.14955)
 		(stroke
 			(width 0.2)
@@
 	)
 	(gr_arc
-		(start 136.5 108.75)
-		(mid 135.914214 110.164214)
-		(end 134.5 110.75)
+		(start 136.525 108.75)
+		(mid 135.939214 110.164214)
+		(end 134.525 110.75)
 		(stroke
 			(width 0.2)
@@
 	)
 	(gr_circle
-		(center 132.75 107.00015)
-		(end 133.88 108.65015)
+		(center 132.775 107.00015)
+		(end 133.905 108.65015)
 		(stroke
 			(width 0.2)
@@
 	)
 	(gr_circle
-		(center 132.75 64.49985)
-		(end 133.88 66.14985)
+		(center 132.775 64.49985)
+		(end 133.905 66.14985)
 		(stroke
 			(width 0.2)
@@
 	)
 	(segment
-		(start 115.9 63.15)
-		(end 115.9 63.175)
-		(width 0.2)
-		(layer "B.Cu")
-		(net 1)
-	)
-	(segment
 		(start 128.675 66.3)
 		(end 127 66.3)
@@
 	)
 	(segment
-		(start 117.04 74.5)
-		(end 117.04 73.6615)
+		(start 117.04 77.5)
+		(end 117 77.5)
 		(width 0.5)
 		(layer "B.Cu")
@@
 	)
 	(segment
+		(start 117 77.5)
+		(end 114.5 80)
+		(width 0.5)
+		(layer "B.Cu")
+		(net 12)
+	)
+	(segment
 		(start 117.04 74.5)
 		(end 117.04 76)
@@
 	)
 	(segment
+		(start 114.5 80)
+		(end 105.5 80)
+		(width 0.5)
+		(layer "B.Cu")
+		(net 12)
+	)
+	(segment
 		(start 105.5115 80)
 		(end 114.445 71.0665)
 		(width 0.5)
-		(layer "B.Cu")
-		(net 12)
-	)
-	(segment
-		(start 117.04 73.6615)
-		(end 114.445 71.0665)
-		(width 0.5)
